File: boards/16buttons/16buttons.kicad_pcb (KiCad board)
At the start: 2 copper layers, 165.1 x 66 mm, 44 parts, among them J1 i2c connector, J2 i2c connector, SW1 SW_Push, SW10 SW_Push, SW11 SW_Push, SW12 SW_Push, SW13 SW_Push, SW14 SW_Push, SW15 SW_Push, SW16 SW_Push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

Commit message: board tweaks before OSH Park order
Parts:
- JP0, JP1, JP2: footprint Jumper:SolderJumper-3_P1.3mm_Bridged12_Pad1.0x1.5mm -> 16buttons:SolderJumper_Bridged12
Routing:
- net /Addr2: track 37.0 -> 34.3 mm
- net /Vin: track 227.4 -> 225.0 mm
- net /Addr1: track 38.5 -> 36.3 mm
- net /SDA: track 204.2 -> 203.7 mm
Other:
- board text added: "Accordion Synth Prototype 4 / skybrian 2020-02"
