File: boards/16buttons/16buttons.sch (KiCad schematic (older format))
At the start: 22 parts, among them J1 i2c connector, J2 i2c connector, SW1 SW_Push, SW10 SW_Push, SW11 SW_Push, SW12 SW_Push, SW13 SW_Push, SW14 SW_Push, SW15 SW_Push, SW16 SW_Push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

Commit message: board tweaks before OSH Park order
Parts:
- JP0, JP1, JP2: footprint Jumper:SolderJumper-3_P1.3mm_Bridged12_Pad1.0x1.5mm -> 16buttons:SolderJumper_Bridged12
Changed lines of the file:
@@
 F 0 "JP2" V 1950 4367 50  0000 L CNN
 F 1 "SolderJumper" V 1905 4368 50  0001 L CNN
-F 2 "Jumper:SolderJumper-3_P1.3mm_Bridged12_Pad1.0x1.5mm" H 1950 4300 50  0001 C CNN
+F 2 "16buttons:SolderJumper_Bridged12" H 1950 4300 50  0001 C CNN
 F 3 "~" H 1950 4300 50  0001 C CNN
 	1    1950 4300
@@
 F 0 "JP1" V 2350 4467 50  0000 L CNN
 F 1 "SolderJumper" V 2305 4468 50  0001 L CNN
-F 2 "Jumper:SolderJumper-3_P1.3mm_Bridged12_Pad1.0x1.5mm" H 2350 4400 50  0001 C CNN
+F 2 "16buttons:SolderJumper_Bridged12" H 2350 4400 50  0001 C CNN
 F 3 "~" H 2350 4400 50  0001 C CNN
 	1    2350 4400
@@
 F 0 "JP0" V 2750 4567 50  0000 L CNN
 F 1 "SolderJumper" V 2705 4568 50  0001 L CNN
-F 2 "Jumper:SolderJumper-3_P1.3mm_Bridged12_Pad1.0x1.5mm" H 2750 4500 50  0001 C CNN
+F 2 "16buttons:SolderJumper_Bridged12" H 2750 4500 50  0001 C CNN
 F 3 "~" H 2750 4500 50  0001 C CNN
 	1    2750 4500
